Commit message: remove namespace

File: vrx_urdf/wamv_description/urdf/thrusters/engine.xacro (robot description, xacro)
@@ -3,5 +3,5 @@
   <!-- Macro for inserting an engine with its propeller. -->
   <xacro:macro name="engine" params="prefix position:='0 0 0' orientation:='0 0 0'">
-    <link name="${namespace}/${prefix}_engine_link">
+    <link name="/${prefix}_engine_link">
       <visual>
         <geometry>
@@ -26,5 +26,5 @@
       </inertial>
     </link>
-    <link name="${namespace}/${prefix}_propeller_link">
+    <link name="/${prefix}_propeller_link">
       <visual>
         <geometry>
@@ -43,15 +43,15 @@
       </inertial>
     </link>
-    <joint name="${namespace}/${prefix}_chassis_engine_joint" type="revolute">
+    <joint name="/${prefix}_chassis_engine_joint" type="revolute">
       <axis xyz="0 0 1"/>
       <limit lower="${-pi}" upper="${pi}" effort="10" velocity="10"/>
       <origin xyz="${position}" rpy="${orientation}"/>
-      <parent link="${namespace}/base_link"/>
-      <child link="${namespace}/${prefix}_engine_link"/>
+      <parent link="/base_link"/>
+      <child link="/${prefix}_engine_link"/>
     </joint>
-    <joint name="${namespace}/${prefix}_engine_propeller_joint" type="continuous">
+    <joint name="/${prefix}_engine_propeller_joint" type="continuous">
       <axis rpy="0 0 0" xyz="1 0 0"/>
-      <parent link="${namespace}/${prefix}_engine_link"/>
-      <child link="${namespace}/${prefix}_propeller_link"/>
+      <parent link="/${prefix}_engine_link"/>
+      <child link="/${prefix}_propeller_link"/>
       <origin rpy="0 0 0" xyz="-0.278156 0 -0.509371"/>
       <limit effort="100" velocity="100" />

File: vrx_urdf/wamv_description/urdf/wamv_base.urdf.xacro (robot description, xacro)
@@ -85,5 +85,5 @@
   </xacro:macro>
   <!-- Basic model of the 16' WAM-V USV -->
-  <link name="${namespace}/base_link">
+  <link name="/base_link">
     <visual>
       <geometry>
@@ -111,5 +111,5 @@
     <enable_wind>true</enable_wind>
   </gazebo>
-  <gazebo reference="${namespace}/base_link">
+  <gazebo reference="/base_link">
     <visual>
       <material>
@@ -129,11 +129,11 @@
       <contact>
         <!-- collisions are renamed during urdf -> sdf fixed joint lumping -->
-        <collision>${namespace}/base_link_fixed_joint_lump__top_base_collision_24</collision>
-        <collision>${namespace}/base_link_fixed_joint_lump__left_float_collision</collision>
-        <collision>${namespace}/base_link_fixed_joint_lump__left_mid_float_collision_1</collision>
-        <collision>${namespace}/base_link_fixed_joint_lump__left_front_float_collision_2</collision>
-        <collision>${namespace}/base_link_fixed_joint_lump__right_float_collision_12</collision>
-        <collision>${namespace}/base_link_fixed_joint_lump__right_mid_float_collision_13</collision>
-        <collision>${namespace}/base_link_fixed_joint_lump__right_front_float_collision_14</collision>
+        <collision>/base_link_fixed_joint_lump__top_base_collision_24</collision>
+        <collision>/base_link_fixed_joint_lump__left_float_collision</collision>
+        <collision>/base_link_fixed_joint_lump__left_mid_float_collision_1</collision>
+        <collision>/base_link_fixed_joint_lump__left_front_float_collision_2</collision>
+        <collision>/base_link_fixed_joint_lump__right_float_collision_12</collision>
+        <collision>/base_link_fixed_joint_lump__right_mid_float_collision_13</collision>
+        <collision>/base_link_fixed_joint_lump__right_front_float_collision_14</collision>
         <topic>/vrx/contacts</topic>
       </contact>

File: vrx_urdf/wamv_gazebo/urdf/components/ball_shooter.xacro (robot description, xacro)
@@ -1,5 +1,5 @@
 <?xml version="1.0"?>
 <robot xmlns:xacro="http://ros.org/wiki/xacro">
-  <xacro:macro name="wamv_ball_shooter" params="name:='ball_shooter' frameId:='wamv/ball_shooter' x:=0.55 y:=0.35 z:=1.4 pitch:='0' yaw:='0'">
+  <xacro:macro name="wamv_ball_shooter" params="name:='ball_shooter' frameId:='/ball_shooter' x:=0.55 y:=0.35 z:=1.4 pitch:='0' yaw:='0'">
     <link name="${namespace}/${name}_base_link">
       <visual>
@@ -96,5 +96,5 @@
           <model_name>blue_projectile</model_name>
           <link_name>link</link_name>
-          <frame>wamv/ball_shooter_launcher_link</frame>
+          <frame>/ball_shooter_launcher_link</frame>
           <pose>0.14 0 0 0 0 0</pose>
         </projectile>

File: vrx_urdf/wamv_gazebo/urdf/components/wamv_p3d.xacro (robot description, xacro)
@@ -9,5 +9,5 @@
         <odom_publish_frequency>10.0</odom_publish_frequency>
         <odom_frame>map</odom_frame>
-        <robot_base_frame>wamv/base_link</robot_base_frame>
+        <robot_base_frame>/base_link</robot_base_frame>
       </plugin>
     </gazebo>
